Commit message: meshをvisualとcollisionに分けた（暫定版モデル）

File: crane_x7_description/urdf/crane_x7.urdf (robot description, URDF)
Before this commit: robot crane_x7, 20 links, 19 joints
Links:
- link HAND_A: geometry collision mesh filename=package://crane_x7_description/meshes/collision/HandA.stl scale=1.0 1.0 1.0; visual mesh filename=package://crane_x7_description/meshes/visual/HandA.stl scale=1.0 1.0 1.0
- link HAND_B: geometry collision mesh filename=package://crane_x7_description/meshes/collision/HandB.stl scale=1.0 1.0 1.0; visual mesh filename=package://crane_x7_description/meshes/visual/HandB.stl scale=1.0 1.0 1.0
- link LINK1: geometry collision mesh filename=package://crane_x7_description/meshes/collision/Link1.stl scale=1.0 1.0 1.0; visual mesh filename=package://crane_x7_description/meshes/visual/Link1.stl scale=1.0 1.0 1.0
- link LINK2: geometry collision mesh filename=package://crane_x7_description/meshes/collision/Link2.stl scale=1.0 1.0 1.0; visual mesh filename=package://crane_x7_description/meshes/visual/Link2.stl scale=1.0 1.0 1.0
- link LINK2_COVER_L: geometry collision mesh filename=package://crane_x7_description/meshes/collision/Link_Cover.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 scale=1.0 1.0 1.0; visual mesh filename=package://crane_x7_description/meshes/visual/Link_Cover.stl scale=1.0 1.0 1.0
- link LINK2_COVER_R: geometry collision mesh filename=package://crane_x7_description/meshes/collision/Link_Cover.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 scale=1.0 1.0 1.0; visual mesh filename=package://crane_x7_description/meshes/visual/Link_Cover.stl scale=1.0 1.0 1.0
- link LINK3: geometry collision mesh filename=package://crane_x7_description/meshes/collision/Link3.stl scale=1.0 1.0 1.0; visual mesh filename=package://crane_x7_description/meshes/visual/Link3.stl scale=1.0 1.0 1.0
- link LINK4: geometry collision mesh filename=package://crane_x7_description/meshes/collision/Link4.stl scale=1.0 1.0 1.0; visual mesh filename=package://crane_x7_description/meshes/visual/Link4.stl scale=1.0 1.0 1.0
- link LINK4_COVER_L: geometry collision mesh filename=package://crane_x7_description/meshes/collision/Link_Cover.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 scale=1.0 1.0 1.0; visual mesh filename=package://crane_x7_description/meshes/visual/Link_Cover.stl scale=1.0 1.0 1.0
- link LINK4_COVER_R: geometry collision mesh filename=package://crane_x7_description/meshes/collision/Link_Cover.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 scale=1.0 1.0 1.0; visual mesh filename=package://crane_x7_description/meshes/visual/Link_Cover.stl scale=1.0 1.0 1.0
- link LINK5: geometry collision mesh filename=package://crane_x7_description/meshes/collision/Link5.stl scale=1.0 1.0 1.0; visual mesh filename=package://crane_x7_description/meshes/visual/Link5.stl scale=1.0 1.0 1.0
- link LINK5_LOGO_CORP_L: geometry collision mesh filename=package://crane_x7_description/meshes/collision/Logo_Corp.s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 scale=1.0 1.0 1.0; visual mesh filename=package://crane_x7_description/meshes/visual/Logo_Corp.stl scale=1.0 1.0 1.0
- link LINK5_LOGO_CORP_R: geometry collision mesh filename=package://crane_x7_description/meshes/collision/Logo_Corp.s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 scale=1.0 1.0 1.0; visual mesh filename=package://crane_x7_description/meshes/visual/Logo_Corp.stl scale=1.0 1.0 1.0
- link LINK5_LOGO_RABBIT_L: geometry collision mesh filename=package://crane_x7_description/meshes/collision/Logo_Rabbit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 scale=1.0 1.0 1.0; visual mesh filename=package://crane_x7_description/meshes/visual/Logo_Rabbit.stl scale=1.0 1.0 1.0
- link LINK5_LOGO_RABBIT_R: geometry collision mesh filename=package://crane_x7_description/meshes/collision/Logo_Rabbit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 scale=1.0 1.0 1.0; visual mesh filename=package://crane_x7_description/meshes/visual/Logo_Rabbit.stl scale=1.0 1.0 1.0
- link LINK6: geometry collision mesh filename=package://crane_x7_description/meshes/collision/Link6.stl scale=1.0 1.0 1.0; visual mesh filename=package://crane_x7_description/meshes/visual/Link6.stl scale=1.0 1.0 1.0
- link LINK7: geometry collision mesh filename=package://crane_x7_description/meshes/collision/Link7.stl scale=1.0 1.0 1.0; visual mesh filename=package://crane_x7_description/meshes/visual/Link7.stl scale=1.0 1.0 1.0
- link base_frame_link: geometry collision mesh filename=package://crane_x7_description/meshes/collision/Base_Frame.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 scale=1.0 1.0 1.0; visual mesh filename=package://crane_x7_description/meshes/visual/Base_Frame.stl scale=1.0 1.0 1.0
- link base_link: geometry collision mesh filename=package://crane_x7_description/meshes/collision/Base.stl scale=1.0 1.0 1.0; visual mesh filename=package://crane_x7_description/meshes/visual/Base.stl scale=1.0 1.0 1.0
