Commit message: Fix incorrect link names and missing parameters

File: crane_x7_description/urdf/crane_x7.urdf.xacro (robot description, xacro)
@@ -14,18 +14,19 @@
        allows accessing different operational areas, e.g. left-handed vs.
        right-handed robots. -->
-  <crane_plus parent="base_link"
-              base_color="blue"
-              link_1_color="black"
-              link_2_color="black"
-              link_3_color="black"
-              link_4_color="black"
-              link_5_color="black"
-              link_6_color="black"
-              link_7_color="blue"
-              link_cover_color="blue"
+  <crane_x7 parent="base_link"
+              base_color="black"
+              shoulder_color="blue"
+              shoulder_joint_cover_color="red"
+              upper_arm_upper_color="green"
+              upper_arm_lower_color="white"
+              elbow_joint_cover_color="blue"
+              lower_arm_upper_color="red"
+              lower_arm_lower_color="green"
+              wrist_color="white"
               hand_color="blue"
               joints_vlimit="1.571"
-              pan_llimit="-2.617" pan_ulimit="2.617">
+              shoulder_llimit="-2.617"
+              shoulder_ulimit="2.617">
     <origin xyz="0 0 0"/>
-  </crane_plus>
+  </crane_x7>
 </robot>

File: crane_x7_description/urdf/crane_x7.xacro (robot description, xacro)
@@ -3,22 +3,22 @@
   <xacro:include filename="$(find crane_x7_description)/urdf/crane_x7_mounting_plate.xacro"/>
   <xacro:include filename="$(find crane_x7_description)/urdf/crane_x7_arm.xacro"/>
-  <xacro:include filename="$(find crane_x7_description)/urdf/crane_x7_wide_two_finger_hand.xacro"/>
+  <xacro:include filename="$(find crane_x7_description)/urdf/crane_x7_wide_two_finger_gripper.xacro"/>
   <material name="black">
-    <color rgba="0.1 0.1 0.1"/>
+    <color rgba="0.2 0.2 0.2 1.0"/>
   </material>
   <material name="white">
-    <color rgba="0.9 0.9 0.9"/>
+    <color rgba="0.95 0.95 0.95 1.0"/>
   </material>
   <material name="silver">
-    <color rgba="0.5 0.5 0.5"/>
+    <color rgba="0.75 0.75 0.75 1.0"/>
   </material>
   <material name="red">
-    <color rgba="1 0 0"/>
+    <color rgba="1.0 0.0 0.0 1.0"/>
   </material>
   <material name="green">
-    <color rgba="0 1 0"/>
+    <color rgba="0.0 1.0 0.0 1.0"/>
   </material>
   <material name="blue">
-    <color rgba="0 0 1"/>
+    <color rgba="0.0 0.0 1.0 1.0"/>
   </material>
   <xacro:macro name="crane_x7"
@@ -35,6 +35,7 @@
               hand_color
               joints_vlimit
-              pan_llimit
-              pan_ulimit">
+              shoulder_llimit
+              shoulder_ulimit
+              *origin">
     <!-- Mounting plate
          (Root of the manipulator's TF tree) -->
@@ -43,28 +44,31 @@
         name="crane_x7_mounting_plate"
         color="silver">
-      <origin xyz="0 0 0" rpy="0 0 0"/>
+      <xacro:insert_block name="origin"/>
     </crane_x7_mounting_plate>
     <!-- Arm -->
     <crane_x7_arm
         parent="crane_x7_mounting_plate_link"
-        attached_link="crane_x7_gripper_base_link"
+        end_effector_base_link="crane_x7_gripper_base_link"
         base_color="${base_color}"
         shoulder_color="${shoulder_color}"
         shoulder_joint_cover_color="${shoulder_joint_cover_color}"
+        upper_arm_upper_color="${upper_arm_lower_color}"
         upper_arm_lower_color="${upper_arm_lower_color}"
-        upper_arm_lower_color="${upper_arm_lower_color}"
+        elbow_joint_cover_color="${elbow_joint_cover_color}"
         lower_arm_upper_color="${lower_arm_upper_color}"
         lower_arm_lower_color="${lower_arm_lower_color}"
         wrist_color="${wrist_color}"
         joints_vlimit="${joints_vlimit}"
-        pan_llimit="${pan_llimit}"
-        pan_ulimit="${pan_ulimit}">
+        shoulder_llimit="${shoulder_llimit}"
+        shoulder_ulimit="${shoulder_ulimit}">
       <origin xyz="0 0 0" rpy="0 0 0"/>
     </crane_x7_arm>
     <!-- End effector -->
     <crane_x7_wide_two_finger_gripper
-        parent="crane_x7_wrist_link"
         name="crane_x7_gripper"
-        color="${hand_color}">
+        color="${hand_color}"
+        vlimit="${joints_vlimit}"
+        llimit="${M_PI/2}"
+        ulimit="${M_PI/2}">
       <origin xyz="0 0 0" rpy="0 0 0"/>
     </crane_x7_wide_two_finger_gripper>

File: crane_x7_description/urdf/crane_x7_arm.xacro (robot description, xacro)
@@ -1,5 +1,9 @@
 <?xml version="1.0"?>
 <robot xmlns:xacro="http://ros.org/wiki/xacro">
-  <xacro:include filename="$(find crane_x7_description)/urdf/crane_x7_arm_hardware.xacro"/>
+  <xacro:property name="M_PI" value="3.14159"/>
+  <xacro:property name="SCALE_MM" value="0.001"/>
+  <xacro:property name="SCALE_CM" value="0.01"/>
+  <xacro:property name="BASE_FIXED_PART_HEIGHT" value="0.005"/>
+  <!-- Macro for the standard CRANE X7 configuration -->
   <xacro:macro name="crane_x7_arm"
       params="parent
@@ -16,17 +20,21 @@
               joints_vlimit
               shoulder_llimit
-              shoulder_ulimit">
+              shoulder_ulimit
+              *origin">
     <!-- Shoulder -->
-    <crane_x7_shoulder
+    <crane_x7_base
         parent="${parent}"
         name="crane_x7_shoulder"
         fixed_part_color="${base_color}"
+        pan_vlimit="${joints_vlimit}"
+        pan_llimit="${shoulder_llimit}"
+        pan_ulimit="${shoulder_ulimit}"
         revolute_part_color="${shoulder_color}"
-        vlimit="${joints_vlimit}"
-        llimit="${shoulder_llimit}"
-        ulimit="${shoulder_ulimit}"
+        tilt_vlimit="${joints_vlimit}"
+        tilt_llimit="${M_PI/2}"
+        tilt_ulimit="${M_PI/2}"
         attached_link="crane_x7_upper_arm_fixed_part_link">
-      <origin xyz="0 0 0" rpy="0 0 0"/>
-    </crane_x7_shoulder>
+      <xacro:insert_block name="origin"/>
+    </crane_x7_base>
     <!-- Upper arm -->
     <crane_x7_type_1_rotating_link
@@ -45,5 +53,5 @@
     </crane_x7_type_1_rotating_link>
     <!-- Lower arm -->
-    <crane_x7_lower_arm
+    <crane_x7_type_2_rotating_link
         name="crane_x7_lower_arm"
         fixed_part_color="${lower_arm_upper_color}"
@@ -58,7 +66,7 @@
         attached_link="crane_x7_wrist_link">
       <origin xyz="0 0 0" rpy="0 0 0"/>
-    </crane_x7_effector_link_upper>
+    </crane_x7_type_2_rotating_link>
     <!-- Wrist -->
-    <crane_x7_effector_link
+    <crane_x7_wrist
         name="crane_x7_wrist"
         color="${wrist_color}"
@@ -68,4 +76,375 @@
         attached_link="${end_effector_base_link}">
       <origin xyz="0 0 0" rpy="0 0 0"/>
-    </crane_x7_effector_link>
+    </crane_x7_wrist>
+  </xacro:macro>
+  <!-- Composite parts -->
+  <!-- Base pan/tilt-like joint -->
+  <xacro:macro name="crane_x7_base"
+      params="parent name
+      fixed_part_color pan_vlimit pan_llimit pan_ulimit
+      revolute_part_color tilt_vlimit tilt_llimit tilt_ulimit attached_link *origin">
+    <crane_x7_base_fixed_part
+        parent="${parent}"
+        name="${name}_fixed_part"
+        color="${fixed_part_color}"
+        vlimit="${pan_vlimit}"
+        llimit="${pan_llimit}"
+        ulimit="${pan_ulimit}"
+        attached_link="${name}_revolute_part_link">
+      <xacro:insert_block name="origin"/>
+    </crane_x7_base_fixed_part>
+    <crane_x7_base_revolute_part
+        name="${name}_revolute_part"
+        color="${revolute_part_color}"
+        vlimit="${tilt_vlimit}"
+        llimit="${tilt_llimit}"
+        ulimit="${tilt_ulimit}"
+        attached_link="${attached_link}">
+      <xacro:insert_block name="origin"/>
+    </crane_x7_base_revolute_part>
+  </xacro:macro>
+  <!-- Long link with twist capability -->
+  <xacro:macro name="crane_x7_type_1_rotating_link"
+      params="name
+      fixed_part_color fixed_vlimit fixed_llimit fixed_ulimit
+      revolute_part_color revolute_vlimit revolute_llimit revolute_ulimit
+      joint_cover_color attached_link *origin">
+    <crane_x7_rotating_link_1_fixed_part
+        name="${name}_fixed_part"
+        color="${fixed_part_color}"/>
+    <crane_x7_rotating_link_1_revolute_part
+        parent="${name}_fixed_part_link"
+        name="${name}_revolute_part"
+        color="${revolute_part_color}"
+        rotate_vlimit="${fixed_vlimit}"
+        rotate_llimit="${fixed_llimit}"
+        rotate_ulimit="${fixed_ulimit}"
+        twist_vlimit="${revolute_vlimit}"
+        twist_llimit="${revolute_llimit}"
+        twist_ulimit="${revolute_ulimit}"
+        joint_cover_color="${joint_cover_color}"
+        attached_link="${attached_link}">
+      <xacro:insert_block name="origin"/>
+    </crane_x7_rotating_link_1_revolute_part>
+  </xacro:macro>
+  <!-- Arm-to-wrist link with twist capability -->
+  <xacro:macro name="crane_x7_type_2_rotating_link"
+      params="name
+      fixed_part_color fixed_vlimit fixed_llimit fixed_ulimit
+      revolute_part_color revolute_vlimit revolute_llimit revolute_ulimit
+      joint_cover_color attached_link *origin">
+    <crane_x7_rotating_link_2_fixed_part
+        name="${name}_fixed_part"
+        color="${fixed_part_color}"
+        vlimit="${fixed_vlimit}"
+        llimit="${fixed_llimit}"
+        ulimit="${fixed_ulimit}"
+        attached_link="${name}_revolute_part_link">
+      <xacro:insert_block name="origin"/>
+    </crane_x7_rotating_link_2_fixed_part>
+    <crane_x7_rotating_link_2_revolute_part
+        name="${name}_revolute_part"
+        color="${revolute_part_color}"
+        vlimit="${revolute_vlimit}"
+        llimit="${revolute_llimit}"
+        ulimit="${revolute_ulimit}"
+        joint_cover_color="${joint_cover_color}"
+        attached_link="${attached_link}">
+      <xacro:insert_block name="origin"/>
+    </crane_x7_rotating_link_2_revolute_part>
+  </xacro:macro>
+  <!-- Individual parts -->
+  <!-- Mountable part of base -->
+  <xacro:macro name="crane_x7_base_fixed_part"
+      params="parent name color vlimit llimit ulimit attached_link *origin">
+    <!-- Fixed joint to the mounting point -->
+    <joint name="${name}_mount_joint" type="fixed">
+      <xacro:insert_block name="origin"/>
+      <parent link="${parent}"/>
+      <child link="${name}_link"/>
+    </joint>
+    <!-- Main link -->
+    <link name="${name}_link">
+      <visual>
+        <origin xyz="0 0 0" rpy="0 0 0"/>
+        <geometry>
+          <mesh filename="package://crane_x7_description/meshes/visual/base_fixed_part.stl"
+              scale="1 1 1"/>
+        </geometry>
+        <material name="${color}"/>
+      </visual>
+      <collision>
+        <origin xyz="0 0 0" rpy="0 0 0"/>
+        <geometry>
+          <mesh filename="package://crane_x7_description/meshes/collision/base_fixed_part.stl"
+              scale="1 1 1"/>
+        </geometry>
+      </collision>
+      <inertial>
+        <mass value="0.001"/>
+        <origin xyz="0 0 0" rpy="0 0 0"/>
+        <inertia ixx="1" ixy="0.0" ixz="0.0"
+          iyy="1" iyz="0.0"
+          izz="1"/>
+      </inertial>
+    </link>
+    <!-- Pan joint of the shoulder -->
+    <joint name="${name}_pan_joint" type="revolute">
+      <origin xyz="0 0 0" rpy="0 0 0"/>
+      <axis xyz="0 0 1"/>
+      <limit effort="30" velocity="${vlimit}" lower="${llimit}" upper="${ulimit}"/>
+      <parent link="${name}_link"/>
+      <child link="${attached_link}"/>
+    </joint>
+  </xacro:macro>
+  <!-- Rotated part of base -->
+  <xacro:macro name="crane_x7_base_revolute_part"
+      params="name color vlimit llimit ulimit attached_link *origin">
+    <link name="${name}_link">
+      <visual>
+        <origin xyz="0 0 0" rpy="0 0 0"/>
+        <geometry>
+          <mesh filename="package://crane_x7_description/meshes/visual/base_revolute_part.stl"
+              scale="1 1 1"/>
+        </geometry>
+        <material name="${color}"/>
+      </visual>
+      <collision>
+        <origin xyz="0 0 0" rpy="0 0 0"/>
+        <geometry>
+          <mesh filename="package://crane_x7_description/meshes/collision/base_revolute_part.stl"
+              scale="1 1 1"/>
+        </geometry>
+      </collision>
+      <inertial>
+        <mass value="0.001"/>
+        <origin xyz="0 0 0" rpy="0 0 0"/>
+        <inertia ixx="1" ixy="0.0" ixz="0.0"
+          iyy="1" iyz="0.0"
+          izz="1"/>
+      </inertial>
+    </link>
+    <!-- Tilt joint of the shoulder -->
+    <joint name="${name}_tilt_joint" type="revolute">
+      <xacro:insert_block name="origin"/>
+      <axis xyz="0 1 0"/>
+      <limit effort="30" velocity="${vlimit}" lower="${llimit}" upper="${ulimit}"/>
+      <parent link="${name}_link"/>
+      <child link="${attached_link}"/>
+    </joint>
+  </xacro:macro>
+  <!-- "Fixed" part of long twistable link -->
+  <xacro:macro name="crane_x7_rotating_link_1_fixed_part"
+    params="name color">
+    <link name="${name}_link">
+      <visual>
+        <origin xyz="0 0 0" rpy="0 0 0"/>
+        <geometry>
+          <mesh filename="package://crane_x7_description/meshes/visual/rotating_link_type_1_fixed_part.stl"
+              scale="1 1 1"/>
+        </geometry>
+        <material name="${color}"/>
+      </visual>
+      <collision>
+        <origin xyz="0 0 0" rpy="0 0 0"/>
+        <geometry>
+          <mesh filename="package://crane_x7_description/meshes/collision/rotating_link_type_1_fixed_part.stl"
+              scale="1 1 1"/>
+        </geometry>
+      </collision>
+      <inertial>
+        <mass value="0.001"/>
+        <origin xyz="0 0 0" rpy="0 0 0"/>
+        <inertia ixx="1" ixy="0.0" ixz="0.0"
+          iyy="1" iyz="0.0"
+          izz="1"/>
+      </inertial>
+    </link>
+  </xacro:macro>
+  <!-- Rotating part of long twistable link -->
+  <xacro:macro name="crane_x7_rotating_link_1_revolute_part"
+      params="parent name color rotate_vlimit rotate_llimit rotate_ulimit
+        twist_vlimit twist_llimit twist_ulimit joint_cover_color attached_link *origin">
+    <!-- Joint for rotating around long axis -->
+    <joint name="${name}_twist_joint" type="revolute">
+      <xacro:insert_block name="origin"/>
+      <axis xyz="0 0 1"/>
+      <limit effort="30"
+          velocity="${rotate_vlimit}"
+          lower="${rotate_llimit}"
+          upper="${rotate_ulimit}"/>
+      <parent link="${parent}"/>
+      <child link="${name}_link"/>
+    </joint>
+    <link name="${name}_link">
+      <visual>
+        <origin xyz="0 0 0" rpy="0 0 0"/>
+        <geometry>
+          <mesh filename="package://crane_x7_description/meshes/visual/rotating_link_type_1_revolute_part.stl"
+              scale="1 1 1"/>
+        </geometry>
+        <material name="${color}"/>
+      </visual>
+      <visual>
+        <origin xyz="0 0 0" rpy="0 0 0"/>
+        <geometry>
+          <mesh filename="package://crane_x7_description/meshes/visual/joint_cover.stl"
+              scale="1 1 1"/>
+        </geometry>
+        <material name="${joint_cover_color}"/>
+      </visual>
+      <collision>
+        <origin xyz="0 0 0" rpy="0 0 0"/>
+        <geometry>
+          <mesh filename="package://crane_x7_description/meshes/collision/rotating_link_type_1_revolute_part.stl"
+              scale="1 1 1"/>
+        </geometry>
+      </collision>
+      <collision>
+        <origin xyz="0 0 0" rpy="0 0 0"/>
+        <geometry>
+          <mesh filename="package://crane_x7_description/meshes/collision/joint_cover.stl"
+              scale="1 1 1"/>
+        </geometry>
+      </collision>
+      <inertial>
+        <mass value="0.001"/>
+        <origin xyz="0 0 0" rpy="0 0 0"/>
+        <inertia ixx="1" ixy="0.0" ixz="0.0"
+          iyy="1" iyz="0.0"
+          izz="1"/>
+      </inertial>
+    </link>
+    <!-- Joint for rotating the attached part -->
+    <joint name="${name}_rotate_joint" type="revolute">
+      <xacro:insert_block name="origin"/>
+      <axis xyz="0 0 1"/>
+      <limit effort="30"
+          velocity="${twist_vlimit}"
+          lower="${twist_llimit}"
+          upper="${twist_ulimit}"/>
+      <parent link="${name}_link"/>
+      <child link="${attached_link}"/>
+    </joint>
+  </xacro:macro>
+  <!-- "Fixed" part of arm-to-wrist twistable link -->
+  <xacro:macro name="crane_x7_rotating_link_2_fixed_part"
+      params="name color vlimit llimit ulimit attached_link *origin">
+    <link name="${name}_link">
+      <visual>
+        <origin xyz="0 0 0" rpy="0 0 0"/>
+        <geometry>
+          <mesh filename="package://crane_x7_description/meshes/visual/rotating_link_type_2_fixed_part.stl"
+              scale="1 1 1"/>
+        </geometry>
+        <material name="${color}"/>
+      </visual>
+      <collision>
+        <origin xyz="0 0 0" rpy="0 0 0"/>
+        <geometry>
+          <mesh filename="package://crane_x7_description/meshes/collision/rotating_link_type_2_fixed_part.stl"
+              scale="1 1 1"/>
+        </geometry>
+      </collision>
+      <inertial>
+        <mass value="0.001"/>
+        <origin xyz="0 0 0" rpy="0 0 0"/>
+        <inertia ixx="1" ixy="0.0" ixz="0.0"
+          iyy="1" iyz="0.0"
+          izz="1"/>
+      </inertial>
+    </link>
+    <joint name="${name}_joint" type="revolute">
+      <xacro:insert_block name="origin"/>
+      <axis xyz="0 1 0"/>
+      <limit effort="30" velocity="${vlimit}" lower="${llimit}" upper="${ulimit}"/>
+      <parent link="${name}_link"/>
+      <child link="${attached_link}"/>
+    </joint>
+  </xacro:macro>
+  <!-- Rotating part of arm-to-wrist twistable link -->
+  <xacro:macro name="crane_x7_rotating_link_2_revolute_part"
+      params="name color vlimit llimit ulimit joint_cover_color attached_link *origin">
+    <link name="${name}_link">
+      <visual>
+        <origin xyz="0 0 0" rpy="0 0 0"/>
+        <geometry>
+          <mesh filename="package://crane_x7_description/meshes/visual/rotating_link_type_2_revolute_part.stl"
+              scale="1 1 1"/>
+        </geometry>
+        <material name="${color}"/>
+      </visual>
+      <visual>
+        <origin xyz="0 0 0" rpy="0 0 0"/>
+        <geometry>
+          <mesh filename="package://crane_x7_description/meshes/visual/joint_cover.stl"
+              scale="1 1 1"/>
+        </geometry>
+        <material name="${joint_cover_color}"/>
+      </visual>
+      <collision>
+        <origin xyz="0 0 0" rpy="0 0 0"/>
+        <geometry>
+          <mesh filename="package://crane_x7_description/meshes/collision/rotating_link_type_2_revolute_part.stl"
+              scale="1 1 1"/>
+        </geometry>
+      </collision>
+      <collision>
+        <origin xyz="0 0 0" rpy="0 0 0"/>
+        <geometry>
+          <mesh filename="package://crane_x7_description/meshes/collision/joint_cover.stl"
+              scale="1 1 1"/>
+        </geometry>
+      </collision>
+      <inertial>
+        <mass value="0.001"/>
+        <origin xyz="0 0 0" rpy="0 0 0"/>
+        <inertia ixx="1" ixy="0.0" ixz="0.0"
+          iyy="1" iyz="0.0"
+          izz="1"/>
+      </inertial>
+    </link>
+    <joint name="${name}_joint" type="revolute">
+      <xacro:insert_block name="origin"/>
+      <axis xyz="0 1 0"/>
+      <limit effort="30" velocity="${vlimit}" lower="${llimit}" upper="${ulimit}"/>
+      <parent link="${name}_link"/>
+      <child link="${attached_link}"/>
+    </joint>
+  </xacro:macro>
+  <!-- Wrist (end effector attachment link) -->
+  <xacro:macro name="crane_x7_wrist"
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
File: crane_x7_description/urdf/crane_x7_wide_two_finger_gripper.xacro (robot description, xacro)
@@ -4,5 +4,6 @@
   <xacro:property name="SCALE_MM" value="0.001"/>
   <xacro:property name="SCALE_CM" value="0.01"/>
-  <xacro:macro name="crane_x7_wide_two_finger_gripper" params="name color *origin">
+  <xacro:macro name="crane_x7_wide_two_finger_gripper"
+      params="name color vlimit llimit ulimit *origin">
     <link name="${name}_base_link">
       <visual>
@@ -30,5 +31,5 @@
     </link>
     <joint name="${name}_finger_a_joint" type="revolute">
-      <origin xyz="0 0 0" rpy="0 0 0"
+      <origin xyz="0 0 0" rpy="0 0 0"/>
       <axis xyz="0 0 1"/>
       <limit effort="30" velocity="${vlimit}" lower="${llimit}" upper="${ulimit}"/>
@@ -61,5 +62,5 @@
     </link>
     <joint name="${name}_finger_b_joint" type="revolute">
-      <origin xyz="0 0 0" rpy="0 0 0"
+      <origin xyz="0 0 0" rpy="0 0 0"/>
       <axis xyz="0 0 1"/>
       <limit effort="30" velocity="${vlimit}" lower="${llimit}" upper="${ulimit}"/>
