Commit message: Aligned joints

File: crane_x7_description/urdf/crane_x7.urdf.xacro (robot description, xacro)
@@ -25,7 +25,7 @@
               wrist_color="white"
               hand_color="blue"
-              joints_vlimit="1.571"
-              shoulder_llimit="-2.617"
-              shoulder_ulimit="2.617">
+              joints_vlimit="4.81710873"
+              shoulder_llimit="-2.97132"
+              shoulder_ulimit="2.97132">
     <origin xyz="0 0 0"/>
   </crane_x7>

File: crane_x7_description/urdf/crane_x7.xacro (robot description, xacro)
@@ -14,11 +14,11 @@
   </material>
   <material name="red">
-    <color rgba="1.0 0.0 0.0 1.0"/>
+    <color rgba="1.0 0.3 0.3 1.0"/>
   </material>
   <material name="green">
-    <color rgba="0.0 1.0 0.0 1.0"/>
+    <color rgba="0.3 1.0 0.3 1.0"/>
   </material>
   <material name="blue">
-    <color rgba="0.0 0.0 1.0 1.0"/>
+    <color rgba="0.3 0.3 1.0 1.0"/>
   </material>
   <xacro:macro name="crane_x7"
@@ -62,5 +62,5 @@
         shoulder_llimit="${shoulder_llimit}"
         shoulder_ulimit="${shoulder_ulimit}">
-      <origin xyz="0 0 0" rpy="0 0 0"/>
+      <origin xyz="0 0 ${MOUNTING_PLATE_THICKNESS}" rpy="0 0 0"/>
     </crane_x7_arm>
     <!-- End effector -->
@@ -68,9 +68,5 @@
         name="crane_x7_gripper"
         color="${hand_color}"
-        vlimit="${joints_vlimit}"
-        llimit="${M_PI/2}"
-        ulimit="${M_PI/2}">
-      <origin xyz="0 0 0" rpy="0 0 0"/>
-    </crane_x7_wide_two_finger_gripper>
+        vlimit="${joints_vlimit}"/>
   </xacro:macro>
 </robot>

File: crane_x7_description/urdf/crane_x7_arm.xacro (robot description, xacro)
@@ -32,5 +32,5 @@
         revolute_part_color="${shoulder_color}"
         tilt_vlimit="${joints_vlimit}"
-        tilt_llimit="${M_PI/2}"
+        tilt_llimit="-${M_PI/2}"
         tilt_ulimit="${M_PI/2}"
         attached_link="crane_x7_upper_arm_fixed_part_link">
@@ -41,26 +41,24 @@
         name="crane_x7_upper_arm"
         fixed_part_color="${upper_arm_upper_color}"
-        fixed_vlimit="${joints_vlimit}"
-        fixed_llimit="-${M_PI/2}"
-        fixed_ulimit="${M_PI/2}"
+        twist_vlimit="${joints_vlimit}"
+        twist_llimit="-${M_PI/2}"
+        twist_ulimit="${M_PI/2}"
         revolute_part_color="${upper_arm_lower_color}"
-        revolute_vlimit="${joints_vlimit}"
-        revolute_llimit="-${M_PI/2}"
-        revolute_ulimit="${M_PI/2}"
+        rotate_vlimit="${joints_vlimit}"
+        rotate_llimit="-2.80718"
+        rotate_ulimit="0.04141"
         joint_cover_color="${shoulder_joint_cover_color}"
-        attached_link="crane_x7_lower_arm_fixed_part_link">
-      <origin xyz="0 0 0" rpy="0 0 0"/>
-    </crane_x7_type_1_rotating_link>
+        attached_link="crane_x7_lower_arm_fixed_part_link"/>
     <!-- Lower arm -->
     <crane_x7_type_2_rotating_link
         name="crane_x7_lower_arm"
         fixed_part_color="${lower_arm_upper_color}"
-        fixed_vlimit="${joints_vlimit}"
-        fixed_llimit="-${M_PI/2}"
-        fixed_ulimit="${M_PI/2}"
+        twist_vlimit="${joints_vlimit}"
+        twist_llimit="-2.77343"
+        twist_ulimit="1.51403"
         revolute_part_color="${lower_arm_lower_color}"
-        revolute_vlimit="${joints_vlimit}"
-        revolute_llimit="-${M_PI/2}"
-        revolute_ulimit="${M_PI/2}"
+        rotate_vlimit="${joints_vlimit}"
+        rotate_llimit="-${M_PI/2}"
+        rotate_ulimit="${M_PI/2}"
         joint_cover_color="${elbow_joint_cover_color}"
         attached_link="crane_x7_wrist_link">
@@ -72,6 +70,6 @@
         color="${wrist_color}"
         vlimit="${joints_vlimit}"
-        llimit="-${M_PI/2}"
-        ulimit="${M_PI/2}"
+        llimit="-2.96365"
+        ulimit="2.97132"
         attached_link="${end_effector_base_link}">
       <origin xyz="0 0 0" rpy="0 0 0"/>
@@ -100,14 +98,12 @@
         llimit="${tilt_llimit}"
         ulimit="${tilt_ulimit}"
-        attached_link="${attached_link}">
-      <xacro:insert_block name="origin"/>
-    </crane_x7_base_revolute_part>
+        attached_link="${attached_link}"/>
   </xacro:macro>
   <!-- Long link with twist capability -->
   <xacro:macro name="crane_x7_type_1_rotating_link"
       params="name
-      fixed_part_color fixed_vlimit fixed_llimit fixed_ulimit
-      revolute_part_color revolute_vlimit revolute_llimit revolute_ulimit
-      joint_cover_color attached_link *origin">
+      fixed_part_color twist_vlimit twist_llimit twist_ulimit
+      revolute_part_color rotate_vlimit rotate_llimit rotate_ulimit
+      joint_cover_color attached_link">
     <crane_x7_rotating_link_1_fixed_part
         name="${name}_fixed_part"
@@ -117,27 +113,25 @@
         name="${name}_revolute_part"
         color="${revolute_part_color}"
-        rotate_vlimit="${fixed_vlimit}"
-        rotate_llimit="${fixed_llimit}"
-        rotate_ulimit="${fixed_ulimit}"
-        twist_vlimit="${revolute_vlimit}"
-        twist_llimit="${revolute_llimit}"
-        twist_ulimit="${revolute_ulimit}"
+        twist_vlimit="${twist_vlimit}"
+        twist_llimit="${twist_llimit}"
+        twist_ulimit="${twist_ulimit}"
+        rotate_vlimit="${rotate_vlimit}"
+        rotate_llimit="${rotate_llimit}"
+        rotate_ulimit="${rotate_ulimit}"
         joint_cover_color="${joint_cover_color}"
-        attached_link="${attached_link}">
-      <xacro:insert_block name="origin"/>
-    </crane_x7_rotating_link_1_revolute_part>
+        attached_link="${attached_link}"/>
   </xacro:macro>
   <!-- Arm-to-wrist link with twist capability -->
   <xacro:macro name="crane_x7_type_2_rotating_link"
       params="name
-      fixed_part_color fixed_vlimit fixed_llimit fixed_ulimit
-      revolute_part_color revolute_vlimit revolute_llimit revolute_ulimit
+      fixed_part_color twist_vlimit twist_llimit twist_ulimit
+      revolute_part_color rotate_vlimit rotate_llimit rotate_ulimit
       joint_cover_color attached_link *origin">
     <crane_x7_rotating_link_2_fixed_part
         name="${name}_fixed_part"
         color="${fixed_part_color}"
-        vlimit="${fixed_vlimit}"
-        llimit="${fixed_llimit}"
-        ulimit="${fixed_ulimit}"
+        vlimit="${twist_vlimit}"
+        llimit="${twist_llimit}"
+        ulimit="${twist_ulimit}"
         attached_link="${name}_revolute_part_link">
       <xacro:insert_block name="origin"/>
@@ -146,7 +140,7 @@
         name="${name}_revolute_part"
         color="${revolute_part_color}"
-        vlimit="${revolute_vlimit}"
-        llimit="${revolute_llimit}"
-        ulimit="${revolute_ulimit}"
+        vlimit="${rotate_vlimit}"
+        llimit="${rotate_llimit}"
+        ulimit="${rotate_ulimit}"
         joint_cover_color="${joint_cover_color}"
         attached_link="${attached_link}">
@@ -182,6 +176,6 @@
       </collision>
       <inertial>
-        <mass value="0.001"/>
-        <origin xyz="0 0 0" rpy="0 0 0"/>
+        <mass value="0.387313"/>
+        <origin xyz="-0.00669 0.000049 0.017868" rpy="0 0 0"/>
         <inertia ixx="1" ixy="0.0" ixz="0.0"
           iyy="1" iyz="0.0"
@@ -191,17 +185,18 @@
     <!-- Pan joint of the shoulder -->
     <joint name="${name}_pan_joint" type="revolute">
-      <origin xyz="0 0 0" rpy="0 0 0"/>
+      <origin xyz="0 0 ${BASE_FIXED_PART_JOINT_Z}" rpy="0 0 0"/>
       <axis xyz="0 0 1"/>
-      <limit effort="30" velocity="${vlimit}" lower="${llimit}" upper="${ulimit}"/>
-      <parent link="${name}_link"/>
-      <child link="${attached_link}"/>
-    </joint>
-  </xacro:macro>
+      <limit effort="0.5" velocity="${vlimit}" lower="${llimit}" upper="${ulimit}"/>
+      <parent link="${name}_link"/>
+      <child link="${attached_link}"/>
+    </joint>
+  </xacro:macro>
+  <xacro:property name="BASE_FIXED_PART_JOINT_Z" value="0.041"/>
   <!-- Rotated part of base -->
   <xacro:macro name="crane_x7_base_revolute_part"
-      params="name color vlimit llimit ulimit attached_link *origin">
-    <link name="${name}_link">
-      <visual>
-        <origin xyz="0 0 0" rpy="0 0 0"/>
+      params="name color vlimit llimit ulimit attached_link">
+    <link name="${name}_link">
+      <visual>
+        <origin xyz="0 0 0" rpy="0 0 ${M_PI}"/>
         <geometry>
           <mesh filename="package://crane_x7_description/meshes/visual/base_revolute_part.stl"
@@ -211,5 +206,5 @@
       </visual>
       <collision>
-        <origin xyz="0 0 0" rpy="0 0 0"/>
+        <origin xyz="0 0 0" rpy="0 0 ${M_PI}"/>
         <geometry>
           <mesh filename="package://crane_x7_description/meshes/collision/base_revolute_part.stl"
@@ -218,6 +213,6 @@
       </collision>
       <inertial>
-        <mass value="0.001"/>
-        <origin xyz="0 0 0" rpy="0 0 0"/>
+        <mass value="0.235377"/>
+        <origin xyz="0.000013 -0.000407 0.046345" rpy="0 0 0"/>
         <inertia ixx="1" ixy="0.0" ixz="0.0"
           iyy="1" iyz="0.0"
@@ -227,11 +222,12 @@
     <!-- Tilt joint of the shoulder -->
     <joint name="${name}_tilt_joint" type="revolute">
-      <xacro:insert_block name="origin"/>
+      <origin xyz="0 0 ${BASE_REVOLUTE_PART_JOINT_Z}" rpy="0 0 0"/>
       <axis xyz="0 1 0"/>
-      <limit effort="30" velocity="${vlimit}" lower="${llimit}" upper="${ulimit}"/>
-      <parent link="${name}_link"/>
-      <child link="${attached_link}"/>
-    </joint>
-  </xacro:macro>
+      <limit effort="0.5" velocity="${vlimit}" lower="${llimit}" upper="${ulimit}"/>
+      <parent link="${name}_link"/>
+      <child link="${attached_link}"/>
+    </joint>
+  </xacro:macro>
+  <xacro:property name="BASE_REVOLUTE_PART_JOINT_Z" value="0.064"/>
   <!-- "Fixed" part of long twistable link -->
   <xacro:macro name="crane_x7_rotating_link_1_fixed_part"
@@ -239,5 +235,5 @@
     <link name="${name}_link">
       <visual>
-        <origin xyz="0 0 0" rpy="0 0 0"/>
+        <origin xyz="0 0 0" rpy="${M_PI/2} 0 0"/>
         <geometry>
           <mesh filename="package://crane_x7_description/meshes/visual/rotating_link_type_1_fixed_part.stl"
@@ -247,5 +243,5 @@
       </visual>
       <collision>
-        <origin xyz="0 0 0" rpy="0 0 0"/>
+        <origin xyz="0 0 0" rpy="${M_PI/2} 0 0"/>
         <geometry>
           <mesh filename="package://crane_x7_description/meshes/collision/rotating_link_type_1_fixed_part.stl"
@@ -254,78 +250,80 @@
       </collision>
       <inertial>
-        <mass value="0.001"/>
-        <origin xyz="0 0 0" rpy="0 0 0"/>
-        <inertia ixx="1" ixy="0.0" ixz="0.0"
-          iyy="1" iyz="0.0"
-          izz="1"/>
-      </inertial>
-    </link>
-  </xacro:macro>
+        <mass value="0.120005"/>
+        <origin xyz="0.000036 0.037855 -0.00018" rpy="${M_PI/2} 0 0"/>
+        <inertia ixx="1" ixy="0.0" ixz="0.0"
+          iyy="1" iyz="0.0"
+          izz="1"/>
+      </inertial>
+    </link>
+  </xacro:macro>
+  <xacro:property name="TYPE_1_FIXED_PART_JOINT_Z" value="0.065"/>
   <!-- Rotating part of long twistable link -->
   <xacro:macro name="crane_x7_rotating_link_1_revolute_part"
-      params="parent name color rotate_vlimit rotate_llimit rotate_ulimit
-        twist_vlimit twist_llimit twist_ulimit joint_cover_color attached_link *origin">
-    <!-- Joint for rotating around long axis -->
+      params="parent name color twist_vlimit twist_llimit twist_ulimit
+        rotate_vlimit rotate_llimit rotate_ulimit joint_cover_color attached_link">
+    <!-- Joint for twisting around long axis -->
     <joint name="${name}_twist_joint" type="revolute">
-      <xacro:insert_block name="origin"/>
+      <origin xyz="0 0 ${TYPE_1_FIXED_PART_JOINT_Z}" rpy="0 0 0"/>
       <axis xyz="0 0 1"/>
-      <limit effort="30"
+      <limit effort="0.5"
+          velocity="${twist_vlimit}"
+          lower="${twist_llimit}"
+          upper="${twist_ulimit}"/>
+      <parent link="${parent}"/>
+      <child link="${name}_link"/>
+    </joint>
+    <link name="${name}_link">
+      <visual>
+        <origin xyz="0 0 0" rpy="0 0 0"/>
+        <geometry>
+          <mesh filename="package://crane_x7_description/meshes/visual/rotating_link_type_1_revolute_part.stl"
+              scale="1 1 1"/>
+        </geometry>
+        <material name="${color}"/>
+      </visual>
+      <visual>
+        <origin xyz="0 0 0" rpy="0 0 0"/>
+        <geometry>
+          <mesh filename="package://crane_x7_description/meshes/visual/joint_cover.stl"
+              scale="1 1 1"/>
+        </geometry>
+        <material name="${joint_cover_color}"/>
+      </visual>
+      <collision>
+        <origin xyz="0 0 0" rpy="0 0 0"/>
+        <geometry>
+          <mesh filename="package://crane_x7_description/meshes/collision/rotating_link_type_1_revolute_part.stl"
+              scale="1 1 1"/>
+        </geometry>
+      </collision>
+      <collision>
+        <origin xyz="0 0 0" rpy="0 0 0"/>
+        <geometry>
+          <mesh filename="package://crane_x7_description/meshes/collision/joint_cover.stl"
+              scale="1 1 1"/>
+        </geometry>
+      </collision>
+      <inertial>
+        <mass value="0.340878"/>
+        <origin xyz="-0.011533 0.000021 0.083707" rpy="${M_PI/2} 0 0"/>
+        <inertia ixx="1" ixy="0.0" ixz="0.0"
+          iyy="1" iyz="0.0"
+          izz="1"/>
+      </inertial>
+    </link>
+    <!-- Joint for rotating the attached part -->
+    <joint name="${name}_rotate_joint" type="revolute">
+      <origin xyz="0 0 ${TYPE_1_REVOLUTE_PART_JOINT_Z}" rpy="0 0 0"/>
+      <axis xyz="0 -1 0"/>
+      <limit effort="0.5"
           velocity="${rotate_vlimit}"
           lower="${rotate_llimit}"
           upper="${rotate_ulimit}"/>
-      <parent link="${parent}"/>
-      <child link="${name}_link"/>
-    </joint>
-    <link name="${name}_link">
-      <visual>
-        <origin xyz="0 0 0" rpy="0 0 0"/>
-        <geometry>
-          <mesh filename="package://crane_x7_description/meshes/visual/rotating_link_type_1_revolute_part.stl"
-              scale="1 1 1"/>
-        </geometry>
-        <material name="${color}"/>
-      </visual>
-      <visual>
-        <origin xyz="0 0 0" rpy="0 0 0"/>
-        <geometry>
-          <mesh filename="package://crane_x7_description/meshes/visual/joint_cover.stl"
-              scale="1 1 1"/>
-        </geometry>
-        <material name="${joint_cover_color}"/>
-      </visual>
-      <collision>
-        <origin xyz="0 0 0" rpy="0 0 0"/>
-        <geometry>
-          <mesh filename="package://crane_x7_description/meshes/collision/rotating_link_type_1_revolute_part.stl"
-              scale="1 1 1"/>
-        </geometry>
-      </collision>
-      <collision>
-        <origin xyz="0 0 0" rpy="0 0 0"/>
-        <geometry>
-          <mesh filename="package://crane_x7_description/meshes/collision/joint_cover.stl"
-              scale="1 1 1"/>
-        </geometry>
-      </collision>
-      <inertial>
-        <mass value="0.001"/>
-        <origin xyz="0 0 0" rpy="0 0 0"/>
-        <inertia ixx="1" ixy="0.0" ixz="0.0"
-          iyy="1" iyz="0.0"
-          izz="1"/>
-      </inertial>
-    </link>
-    <!-- Joint for rotating the attached part -->
-    <joint name="${name}_rotate_joint" type="revolute">
-      <xacro:insert_block name="origin"/>
-      <axis xyz="0 0 1"/>
-      <limit effort="30"
-          velocity="${twist_vlimit}"
-          lower="${twist_llimit}"
-          upper="${twist_ulimit}"/>
-      <parent link="${name}_link"/>
-      <child link="${attached_link}"/>
-    </joint>
-  </xacro:macro>
+      <parent link="${name}_link"/>
+      <child link="${attached_link}"/>
+    </joint>
+  </xacro:macro>
+  <xacro:property name="TYPE_1_REVOLUTE_PART_JOINT_Z" value="0.185"/>
   <!-- "Fixed" part of arm-to-wrist twistable link -->
   <xacro:macro name="crane_x7_rotating_link_2_fixed_part"
@@ -333,5 +331,5 @@
     <link name="${name}_link">
       <visual>
-        <origin xyz="0 0 0" rpy="0 0 0"/>
+        <origin xyz="0 0 0" rpy="${M_PI/2} 0 0"/>
         <geometry>
           <mesh filename="package://crane_x7_description/meshes/visual/rotating_link_type_2_fixed_part.stl"
@@ -341,5 +339,5 @@
       </visual>
       <collision>
-        <origin xyz="0 0 0" rpy="0 0 0"/>
+        <origin xyz="0 0 0" rpy="${M_PI/2} 0 0"/>
         <geometry>
           <mesh filename="package://crane_x7_description/meshes/collision/rotating_link_type_2_fixed_part.stl"
@@ -348,6 +346,6 @@
       </collision>
       <inertial>
-        <mass value="0.001"/>
-        <origin xyz="0 0 0" rpy="0 0 0"/>
+        <mass value="0.230634"/>
+        <origin xyz="-0.008641 0.083071 -0.000086" rpy="${M_PI} 0 0"/>
         <inertia ixx="1" ixy="0.0" ixz="0.0"
           iyy="1" iyz="0.0"
@@ -356,11 +354,12 @@
     </link>
     <joint name="${name}_joint" type="revolute">
-      <xacro:insert_block name="origin"/>
-      <axis xyz="0 1 0"/>
-      <limit effort="30" velocity="${vlimit}" lower="${llimit}" upper="${ulimit}"/>
-      <parent link="${name}_link"/>
-      <child link="${attached_link}"/>
-    </joint>
-  </xacro:macro>
+      <origin xyz="0 0 ${TYPE_2_FIXED_PART_JOINT_Z}" rpy="0 0 0"/>
+      <axis xyz="0 0 1"/>
+      <limit effort="0.5" velocity="${vlimit}" lower="${llimit}" upper="${ulimit}"/>
+      <parent link="${name}_link"/>
+      <child link="${attached_link}"/>
+    </joint>
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
File: crane_x7_description/urdf/crane_x7_mounting_plate.xacro (robot description, xacro)
@@ -29,8 +29,9 @@
       <inertial>
         <mass value="0.001"/>
-        <origin xyz="0 0 0" rpy="0 0 0"/>
-        <inertia ixx="1" ixy="0.0" ixz="0.0"
-          iyy="1" iyz="0.0"
-          izz="1"/>
+        <origin xyz="-0.00669 0.000049 0.017868" rpy="0 0 0"/>
+        <inertia ixx="1.0" ixy="0.0" ixz="0.0"
+          iyy="1.0" iyz="0.0"
+          izz="1.0"/>
+        <mass value="0.387313"/>
       </inertial>
     </link>

File: crane_x7_description/urdf/crane_x7_wide_two_finger_gripper.xacro (robot description, xacro)
@@ -5,5 +5,5 @@
   <xacro:property name="SCALE_CM" value="0.01"/>
   <xacro:macro name="crane_x7_wide_two_finger_gripper"
-      params="name color vlimit llimit ulimit *origin">
+    params="name color vlimit">
     <link name="${name}_base_link">
       <visual>
@@ -23,6 +23,6 @@
       </collision>
       <inertial>
-        <mass value="0.001"/>
-        <origin xyz="0 0 0" rpy="0 0 0"/>
+        <mass value="0.119807"/>
+        <origin xyz="0.000425 -0.000896 0.018691" rpy="0 0 0"/>
         <inertia ixx="1" ixy="0.0" ixz="0.0"
           iyy="1" iyz="0.0"
@@ -31,7 +31,7 @@
     </link>
     <joint name="${name}_finger_a_joint" type="revolute">
-      <origin xyz="0 0 0" rpy="0 0 0"/>
-      <axis xyz="0 0 1"/>
-      <limit effort="30" velocity="${vlimit}" lower="${llimit}" upper="${ulimit}"/>
+      <origin xyz="-0.012 0.0 0.024" rpy="0 0 0"/>
+      <axis xyz="0 -1 0"/>
+      <limit effort="0.5" velocity="${vlimit}" lower="0.0046" upper="1.62601"/>
       <parent link="${name}_base_link"/>
       <child link="${name}_finger_a_link"/>
@@ -39,5 +39,5 @@
     <link name="${name}_finger_a_link">
       <visual>
-        <origin xyz="0 0 0" rpy="0 0 0"/>
+        <origin xyz="0 0 0" rpy="${M_PI/2} 0 0"/>
         <geometry>
           <mesh filename="package://crane_x7_description/meshes/visual/wide_two_finger_gripper_finger_a.stl"
@@ -54,6 +54,6 @@
       </collision>
       <inertial>
-        <mass value="0.001"/>
-        <origin xyz="0 0 0" rpy="0 0 0"/>
+        <mass value="0.015617"/>
+        <origin xyz="-0.002987 0.030318 0.003073" rpy="${M_PI/2} 0 0"/>
         <inertia ixx="1" ixy="0.0" ixz="0.0"
           iyy="1" iyz="0.0"
@@ -62,13 +62,14 @@
     </link>
     <joint name="${name}_finger_b_joint" type="revolute">
-      <origin xyz="0 0 0" rpy="0 0 0"/>
-      <axis xyz="0 0 1"/>
-      <limit effort="30" velocity="${vlimit}" lower="${llimit}" upper="${ulimit}"/>
+      <origin xyz="0.012 0.0 0.024" rpy="0 0 0"/>
+      <axis xyz="0 1 0"/>
+      <limit effort="0.5" velocity="${vlimit}" lower="0.0046" upper="1.62601"/>
       <parent link="${name}_base_link"/>
       <child link="${name}_finger_b_link"/>
+      <mimic joint="${name}_finger_a_joint"/>
     </joint>
     <link name="${name}_finger_b_link">
       <visual>
-        <origin xyz="0 0 0" rpy="0 0 0"/>
+        <origin xyz="0 0 0" rpy="${M_PI/2} 0 0"/>
         <geometry>
           <mesh filename="package://crane_x7_description/meshes/visual/wide_two_finger_gripper_finger_b.stl"
@@ -85,6 +86,6 @@
       </collision>
       <inertial>
-        <mass value="0.001"/>
-        <origin xyz="0 0 0" rpy="0 0 0"/>
+        <mass value="0.014417"/>
+        <origin xyz="0.003058 0.031215 0.002548" rpy="${M_PI/2} 0 0"/>
         <inertia ixx="1" ixy="0.0" ixz="0.0"
           iyy="1" iyz="0.0"
