Commit message: Finished URDF

File: crane_x7_description/urdf/crane_x7.urdf.xacro (robot description, xacro)
@@ -15,17 +15,18 @@
        right-handed robots. -->
   <crane_x7 parent="base_link"
-              base_color="black"
-              shoulder_color="blue"
+              base_color="red"
+              shoulder_color="white"
               shoulder_joint_cover_color="red"
-              upper_arm_upper_color="green"
+              upper_arm_upper_color="white"
               upper_arm_lower_color="white"
-              elbow_joint_cover_color="blue"
-              lower_arm_upper_color="red"
-              lower_arm_lower_color="green"
+              elbow_joint_cover_color="red"
+              lower_arm_upper_color="white"
+              lower_arm_lower_color="white"
               wrist_color="white"
-              hand_color="blue"
+              hand_color="red"
               joints_vlimit="4.81710873"
               shoulder_llimit="-2.97132"
-              shoulder_ulimit="2.97132">
+              shoulder_ulimit="2.97132"
+              logos_definition="crane_x7_rt_logos.xacro">
     <origin xyz="0 0 0"/>
   </crane_x7>

File: crane_x7_description/urdf/crane_x7.xacro (robot description, xacro)
@@ -37,4 +37,5 @@
               shoulder_llimit
               shoulder_ulimit
+              logos_definition
               *origin">
     <!-- Mounting plate
@@ -61,5 +62,6 @@
         joints_vlimit="${joints_vlimit}"
         shoulder_llimit="${shoulder_llimit}"
-        shoulder_ulimit="${shoulder_ulimit}">
+        shoulder_ulimit="${shoulder_ulimit}"
+        logos_definition="${logos_definition}">
       <origin xyz="0 0 ${MOUNTING_PLATE_THICKNESS}" rpy="0 0 0"/>
     </crane_x7_arm>

File: crane_x7_description/urdf/crane_x7_arm.xacro (robot description, xacro)
@@ -21,4 +21,5 @@
               shoulder_llimit
               shoulder_ulimit
+              logos_definition
               *origin">
     <!-- Shoulder -->
@@ -62,5 +63,6 @@
         rotate_ulimit="${M_PI/2}"
         joint_cover_color="${elbow_joint_cover_color}"
-        attached_link="crane_x7_wrist_link">
+        attached_link="crane_x7_wrist_link"
+        logos_definition="${logos_definition}">
       <origin xyz="0 0 0" rpy="0 0 0"/>
     </crane_x7_type_2_rotating_link>
@@ -108,5 +110,6 @@
     <crane_x7_rotating_link_1_fixed_part
         name="${name}_fixed_part"
-        color="${fixed_part_color}"/>
+        color="${fixed_part_color}"
+        joint_cover_color="${joint_cover_color}"/>
     <crane_x7_rotating_link_1_revolute_part
         parent="${name}_fixed_part_link"
@@ -119,5 +122,4 @@
         rotate_llimit="${rotate_llimit}"
         rotate_ulimit="${rotate_ulimit}"
-        joint_cover_color="${joint_cover_color}"
         attached_link="${attached_link}"/>
   </xacro:macro>
@@ -127,5 +129,5 @@
       fixed_part_color twist_vlimit twist_llimit twist_ulimit
       revolute_part_color rotate_vlimit rotate_llimit rotate_ulimit
-      joint_cover_color attached_link *origin">
+      joint_cover_color attached_link logos_definition *origin">
     <crane_x7_rotating_link_2_fixed_part
         name="${name}_fixed_part"
@@ -134,4 +136,5 @@
         llimit="${twist_llimit}"
         ulimit="${twist_ulimit}"
+        joint_cover_color="${joint_cover_color}"
         attached_link="${name}_revolute_part_link">
       <xacro:insert_block name="origin"/>
@@ -143,6 +146,6 @@
         llimit="${rotate_llimit}"
         ulimit="${rotate_ulimit}"
-        joint_cover_color="${joint_cover_color}"
-        attached_link="${attached_link}">
+        attached_link="${attached_link}"
+        logos_definition="${logos_definition}">
       <xacro:insert_block name="origin"/>
     </crane_x7_rotating_link_2_revolute_part>
@@ -232,5 +235,5 @@
   <!-- "Fixed" part of long twistable link -->
   <xacro:macro name="crane_x7_rotating_link_1_fixed_part"
-    params="name color">
+    params="name color joint_cover_color">
     <link name="${name}_link">
       <visual>
@@ -257,4 +260,64 @@
       </inertial>
     </link>
+    <!-- Joint covers -->
+    <!-- TODO: Once rviz fixes its multi-material display bug, move these into the parent link -->
+    <link name="${name}_joint_cover_l_link">
+      <visual>
+        <origin xyz="0 0 0" rpy="-${M_PI/2} 0 0"/>
+        <geometry>
+          <mesh filename="package://crane_x7_description/meshes/visual/joint_cover.stl"
+              scale="1 1 1"/>
+        </geometry>
+        <material name="${joint_cover_color}"/>
+      </visual>
+      <collision>
+        <origin xyz="0 0 0" rpy="0 0 0"/>
+        <geometry>
+          <mesh filename="package://crane_x7_description/meshes/collision/joint_cover.stl"
+              scale="1 1 1"/>
+        </geometry>
+      </collision>
+      <inertial>
+        <mass value="0.005"/>
+        <origin xyz="0.000036 0.037855 -0.00018" rpy="${M_PI/2} 0 0"/>
+        <inertia ixx="1" ixy="0.0" ixz="0.0"
+          iyy="1" iyz="0.0"
+          izz="1"/>
+      </inertial>
+    </link>
+    <joint name="${name}_joint_cover_l_joint" type="fixed">
+      <parent link="${name}_link"/>
+      <child link="${name}_joint_cover_l_link"/>
+      <origin xyz="0 0.0316 0" rpy="0 0 0"/>
+    </joint>
+    <link name="${name}_joint_cover_r_link">
+      <visual>
+        <origin xyz="0 0 0" rpy="${M_PI/2} 0 0"/>
+        <geometry>
+          <mesh filename="package://crane_x7_description/meshes/visual/joint_cover.stl"
+              scale="1 1 1"/>
+        </geometry>
+        <material name="${joint_cover_color}"/>
+      </visual>
+      <collision>
+        <origin xyz="0 0 0" rpy="0 0 0"/>
+        <geometry>
+          <mesh filename="package://crane_x7_description/meshes/collision/joint_cover.stl"
+              scale="1 1 1"/>
+        </geometry>
+      </collision>
+      <inertial>
+        <mass value="0.005"/>
+        <origin xyz="0.000036 0.037855 -0.00018" rpy="${M_PI/2} 0 0"/>
+        <inertia ixx="1" ixy="0.0" ixz="0.0"
+          iyy="1" iyz="0.0"
+          izz="1"/>
+      </inertial>
+    </link>
+    <joint name="${name}_joint_cover_r_joint" type="fixed">
+      <parent link="${name}_link"/>
+      <child link="${name}_joint_cover_r_link"/>
+      <origin xyz="0 -0.0316 0" rpy="0 0 0"/>
+    </joint>
   </xacro:macro>
   <xacro:property name="TYPE_1_FIXED_PART_JOINT_Z" value="0.065"/>
@@ -262,5 +325,5 @@
   <xacro:macro name="crane_x7_rotating_link_1_revolute_part"
       params="parent name color twist_vlimit twist_llimit twist_ulimit
-        rotate_vlimit rotate_llimit rotate_ulimit joint_cover_color attached_link">
+        rotate_vlimit rotate_llimit rotate_ulimit attached_link">
     <!-- Joint for twisting around long axis -->
     <joint name="${name}_twist_joint" type="revolute">
@@ -283,23 +346,8 @@
         <material name="${color}"/>
       </visual>
-      <visual>
-        <origin xyz="0 0 0" rpy="0 0 0"/>
-        <geometry>
-          <mesh filename="package://crane_x7_description/meshes/visual/joint_cover.stl"
-              scale="1 1 1"/>
-        </geometry>
-        <material name="${joint_cover_color}"/>
-      </visual>
       <collision>
         <origin xyz="0 0 0" rpy="0 0 0"/>
         <geometry>
           <mesh filename="package://crane_x7_description/meshes/collision/rotating_link_type_1_revolute_part.stl"
-              scale="1 1 1"/>
-        </geometry>
-      </collision>
-      <collision>
-        <origin xyz="0 0 0" rpy="0 0 0"/>
-        <geometry>
-          <mesh filename="package://crane_x7_description/meshes/collision/joint_cover.stl"
               scale="1 1 1"/>
         </geometry>
@@ -328,5 +376,5 @@
   <!-- "Fixed" part of arm-to-wrist twistable link -->
   <xacro:macro name="crane_x7_rotating_link_2_fixed_part"
-      params="name color vlimit llimit ulimit attached_link *origin">
+      params="name color vlimit llimit ulimit joint_cover_color attached_link *origin">
     <link name="${name}_link">
       <visual>
@@ -360,9 +408,69 @@
       <child link="${attached_link}"/>
     </joint>
+    <!-- Joint covers -->
+    <!-- TODO: Once rviz fixes its multi-material display bug, move these into the parent link -->
+    <link name="${name}_joint_cover_l_link">
+      <visual>
+        <origin xyz="0 0 0" rpy="-${M_PI/2} 0 0"/>
+        <geometry>
+          <mesh filename="package://crane_x7_description/meshes/visual/joint_cover.stl"
+              scale="1 1 1"/>
+        </geometry>
+        <material name="${joint_cover_color}"/>
+      </visual>
+      <collision>
+        <origin xyz="0 0 0" rpy="0 0 0"/>
+        <geometry>
+          <mesh filename="package://crane_x7_description/meshes/collision/joint_cover.stl"
+              scale="1 1 1"/>
+        </geometry>
+      </collision>
+      <inertial>
+        <mass value="0.005"/>
+        <origin xyz="0.000036 0.037855 -0.00018" rpy="${M_PI/2} 0 0"/>
+        <inertia ixx="1" ixy="0.0" ixz="0.0"
+          iyy="1" iyz="0.0"
+          izz="1"/>
+      </inertial>
+    </link>
+    <joint name="${name}_joint_cover_l_joint" type="fixed">
+      <parent link="${name}_link"/>
+      <child link="${name}_joint_cover_l_link"/>
+      <origin xyz="0 0.025 0" rpy="0 0 0"/>
+    </joint>
+    <link name="${name}_joint_cover_r_link">
+      <visual>
+        <origin xyz="0 0 0" rpy="${M_PI/2} 0 0"/>
+        <geometry>
+          <mesh filename="package://crane_x7_description/meshes/visual/joint_cover.stl"
+              scale="1 1 1"/>
+        </geometry>
+        <material name="${joint_cover_color}"/>
+      </visual>
+      <collision>
+        <origin xyz="0 0 0" rpy="0 0 0"/>
+        <geometry>
+          <mesh filename="package://crane_x7_description/meshes/collision/joint_cover.stl"
+              scale="1 1 1"/>
+        </geometry>
+      </collision>
+      <inertial>
+        <mass value="0.005"/>
+        <origin xyz="0.000036 0.037855 -0.00018" rpy="${M_PI/2} 0 0"/>
+        <inertia ixx="1" ixy="0.0" ixz="0.0"
+          iyy="1" iyz="0.0"
+          izz="1"/>
+      </inertial>
+    </link>
+    <joint name="${name}_joint_cover_r_joint" type="fixed">
+      <parent link="${name}_link"/>
+      <child link="${name}_joint_cover_r_link"/>
+      <origin xyz="0 -0.025 0" rpy="0 0 0"/>
+    </joint>
   </xacro:macro>
   <xacro:property name="TYPE_2_FIXED_PART_JOINT_Z" value="0.121"/>
   <!-- Rotating part of arm-to-wrist twistable link -->
   <xacro:macro name="crane_x7_rotating_link_2_revolute_part"
-      params="name color vlimit llimit ulimit joint_cover_color attached_link *origin">
+      params="name color vlimit llimit ulimit attached_link logos_definition *origin">
     <link name="${name}_link">
       <visual>
@@ -374,23 +482,8 @@
         <material name="${color}"/>
       </visual>
-      <visual>
-        <origin xyz="0 0 0" rpy="0 0 0"/>
-        <geometry>
-          <mesh filename="package://crane_x7_description/meshes/visual/joint_cover.stl"
-              scale="1 1 1"/>
-        </geometry>
-        <material name="${joint_cover_color}"/>
-      </visual>
       <collision>
         <origin xyz="0 0 0" rpy="0 0 0"/>
         <geometry>
           <mesh filename="package://crane_x7_description/meshes/collision/rotating_link_type_2_revolute_part.stl"
-              scale="1 1 1"/>
-        </geometry>
-      </collision>
-      <collision>
-        <origin xyz="0 0 0" rpy="0 0 0"/>
-        <geometry>
-          <mesh filename="package://crane_x7_description/meshes/collision/joint_cover.stl"
               scale="1 1 1"/>
         </geometry>
@@ -411,4 +504,8 @@
       <child link="${attached_link}"/>
     </joint>
+    <!-- Logos -->
+    <!-- TODO: Once rviz fixes its multi-material display bug, move these into the parent link -->
+    <xacro:include filename="${logos_definition}"/>
+    <crane_x7_logos parent="${name}_link"/>
   </xacro:macro>
   <xacro:property name="TYPE_2_REVOLUTE_PART_JOINT_Z" value="0.129"/>
