Commit message: Can control crane_x7 in gazebo with MoveIt.

File: crane_x7_description/urdf/crane_x7.urdf.xacro (robot description, xacro)
@@ -10,4 +10,10 @@
   <!-- Link to provide the location reference for the arm -->
   <link name="base_link"/>
+  <!-- Used for fixing robot to Gazebo 'base_link' -->
+  <link name="world"/>
+  <joint name="base_link_to_world_joint" type="fixed">
+    <parent link="world"/>
+    <child link="base_link"/>
+  </joint>
   <!-- Use the crane_x7 macro to configure a Crane X7 arm with desired joint
        velocities limit and lower/upper limits for the first joint. This

File: crane_x7_description/urdf/crane_x7_arm.xacro (robot description, xacro)
@@ -70,9 +70,9 @@
       </collision>
       <inertial>
-        <mass value="0.387313"/>
-        <origin xyz="-0.00669 0.000049 0.017868" rpy="0 0 0"/>
-        <inertia ixx="1" ixy="0.0" ixz="0.0"
-          iyy="1" iyz="0.0"
-          izz="1"/>
+        <mass value="0.388"/>
+        <origin xyz="-6.73E-03 -1.00E-06 1.79E-02" rpy="0 0 0"/>
+        <inertia ixx="3.25E-04" ixy="1.20E-09" ixz="-4.71E-05"
+          iyy="4.83E-04" iyz="1.95E-08"
+          izz="5.86E-04"/>
       </inertial>
     </link>
@@ -81,8 +81,23 @@
       <origin xyz="0 0 0.036" rpy="0 0 0"/>
       <axis xyz="0 0 1"/>
-      <limit effort="0.5" velocity="${joints_vlimit}" lower="${shoulder_llimit}" upper="${shoulder_ulimit}"/>
+      <limit effort="10.0" velocity="${joints_vlimit}" lower="${shoulder_llimit}" upper="${shoulder_ulimit}"/>
       <parent link="${NAME_LINK_BASE}"/>
       <child link="${NAME_LINK_1}"/>
-    </joint>
+      <dynamics damping="0.0" friction="0.0"/>
+    </joint>
+    <!-- For gazebo simulation -->
+    <transmission name="${NAME_JOINT_1}_trans">
+      <provideFeedback>true</provideFeedback>
+      <implicitSpringDamper>0</implicitSpringDamper>
+      <motorTorqueConstant>0.418</motorTorqueConstant>
+      <type>transmission_interface/SimpleTransmission</type>
+      <joint name="${NAME_JOINT_1}">
+        <hardwareInterface>hardware_interface/PositionJointInterface</hardwareInterface>
+      </joint>
+      <actuator name="${NAME_JOINT_1}_motor">
+        <hardwareInterface>hardware_interface/PositionJointInterface</hardwareInterface>
+        <mechanicalReduction>1</mechanicalReduction>
+      </actuator>
+    </transmission>
     <!-- crane_x7_link_1 -->
     <link name="${NAME_LINK_1}">
@@ -103,9 +118,9 @@
       </collision>
       <inertial>
-        <mass value="0.235377"/>
-        <origin xyz="0.000013 -0.000407 0.046345" rpy="0 0 0"/>
-        <inertia ixx="1" ixy="0.0" ixz="0.0"
-          iyy="1" iyz="0.0"
-          izz="1"/>
+        <mass value="0.253"/>
+        <origin xyz="2.43e-04 -1.05E-04 4.70E-02" rpy="0 0 0"/>
+        <inertia ixx="1.79E-04" ixy="-7.32E-08" ixz="8.89E-07"
+          iyy="1.76E-04" iyz="6.23E-07"
+          izz="8.96E-05"/>
       </inertial>
     </link>
@@ -114,8 +129,23 @@
       <origin xyz="0 0 0.064" rpy="0 0 0"/>
       <axis xyz="0 -1 0"/>
-      <limit effort="0.5" velocity="${joints_vlimit}" lower="-${M_PI/2}" upper="${M_PI/2}"/>
+      <limit effort="10.0" velocity="${joints_vlimit}" lower="-${M_PI/2}" upper="${M_PI/2}"/>
       <parent link="${NAME_LINK_1}"/>
       <child link="${NAME_LINK_2}"/>
-    </joint>
+      <dynamics damping="0.0" friction="0.0"/>
+    </joint>
+    <!-- For gazebo simulation -->
+    <transmission name="${NAME_JOINT_2}_trans">
+      <provideFeedback>true</provideFeedback>
+      <implicitSpringDamper>0</implicitSpringDamper>
+      <motorTorqueConstant>0.418</motorTorqueConstant>
+      <type>transmission_interface/SimpleTransmission</type>
+      <joint name="${NAME_JOINT_2}">
+        <hardwareInterface>hardware_interface/PositionJointInterface</hardwareInterface>
+      </joint>
+      <actuator name="${NAME_JOINT_2}_motor">
+        <hardwareInterface>hardware_interface/PositionJointInterface</hardwareInterface>
+        <mechanicalReduction>1</mechanicalReduction>
+      </actuator>
+    </transmission>
     <!-- crane_x7_link_2 -->
     <link name="${NAME_LINK_2}">
@@ -136,9 +166,9 @@
       </collision>
       <inertial>
-        <mass value="0.120005"/>
-        <origin xyz="0.000036 0.037855 -0.00018" rpy="${M_PI/2} 0 0"/>
-        <inertia ixx="1" ixy="0.0" ixz="0.0"
-          iyy="1" iyz="0.0"
-          izz="1"/>
+        <mass value="0.136"/>
+        <origin xyz="3.10E-05 1.90E-05 3.42E-02" rpy="${M_PI/2} 0 0"/>
+        <inertia ixx="1.68E-04" ixy="2.05E-08" ixz="-4.00E-07"
+          iyy="9.62E-05" iyz="6.24E-08"
+          izz="1.34E-04"/>
       </inertial>
     </link>
@@ -166,11 +196,4 @@
         </geometry>
       </collision>
-      <inertial>
-        <mass value="0.005"/>
-        <origin xyz="0.000036 0.037855 -0.00018" rpy="${M_PI/2} 0 0"/>
-        <inertia ixx="1" ixy="0.0" ixz="0.0"
-          iyy="1" iyz="0.0"
-          izz="1"/>
-      </inertial>
     </link>
     <!-- crane_x7_joint_cover_2_r -->
@@ -197,11 +220,4 @@
         </geometry>
       </collision>
-      <inertial>
-        <mass value="0.005"/>
-        <origin xyz="0.000036 0.037855 -0.00018" rpy="${M_PI/2} 0 0"/>
-        <inertia ixx="1" ixy="0.0" ixz="0.0"
-          iyy="1" iyz="0.0"
-          izz="1"/>
-      </inertial>
     </link>
     <!-- crane_x7_joint_3 -->
@@ -209,5 +225,5 @@
       <origin xyz="0 0 0.065" rpy="0 0 0"/>
       <axis xyz="0 0 1"/>
-      <limit effort="0.5"
+      <limit effort="4.0"
           velocity="${joints_vlimit}"
           lower="-${M_PI/2}"
@@ -215,5 +231,20 @@
       <parent link="${NAME_LINK_2}"/>
       <child link="${NAME_LINK_3}"/>
-    </joint>
+      <dynamics damping="0.0" friction="0.0"/>
+    </joint>
+    <!-- For gazebo simulation -->
+    <transmission name="${NAME_JOINT_3}_trans">
+      <provideFeedback>true</provideFeedback>
+      <implicitSpringDamper>0</implicitSpringDamper>
+      <motorTorqueConstant>0.418</motorTorqueConstant>
+      <type>transmission_interface/SimpleTransmission</type>
+      <joint name="${NAME_JOINT_3}">
+        <hardwareInterface>hardware_interface/PositionJointInterface</hardwareInterface>
+      </joint>
+      <actuator name="${NAME_JOINT_3}_motor">
+        <hardwareInterface>hardware_interface/PositionJointInterface</hardwareInterface>
+        <mechanicalReduction>1</mechanicalReduction>
+      </actuator>
+    </transmission>
     <!-- crane_x7_link_3 -->
     <link name="${NAME_LINK_3}">
@@ -234,9 +265,9 @@
       </collision>
       <inertial>
-        <mass value="0.340878"/>
-        <origin xyz="-0.011533 0.000021 0.083707" rpy="${M_PI/2} 0 0"/>
-        <inertia ixx="1" ixy="0.0" ixz="0.0"
-          iyy="1" iyz="0.0"
-          izz="1"/>
+        <mass value="0.321"/>
+        <origin xyz="-1.37E-02 -8.10E-05 9.52E-02" rpy="0 0 0"/>
+        <inertia ixx="1.82E-03" ixy="7.54E-07" ixz="-3.73E-05"
+          iyy="1.88E-03" iyz="4.15E-06"
+          izz="1.59E-04"/>
       </inertial>
     </link>
@@ -245,5 +276,5 @@
       <origin xyz="0 0 0.185" rpy="0 0 0"/>
       <axis xyz="0 -1 0"/>
-      <limit effort="0.5"
+      <limit effort="4.0"
           velocity="${joints_vlimit}"
           lower="-2.80718"
@@ -251,5 +282,20 @@
       <parent link="${NAME_LINK_3}"/>
       <child link="${NAME_LINK_4}"/>
-    </joint>
+      <dynamics damping="0.0" friction="0.0"/>
+    </joint>
+    <!-- For gazebo simulation -->
+    <transmission name="${NAME_JOINT_4}_trans">
+      <provideFeedback>true</provideFeedback>
+      <implicitSpringDamper>0</implicitSpringDamper>
+      <motorTorqueConstant>0.418</motorTorqueConstant>
+      <type>transmission_interface/SimpleTransmission</type>
+      <joint name="${NAME_JOINT_4}">
+        <hardwareInterface>hardware_interface/PositionJointInterface</hardwareInterface>
+      </joint>
+      <actuator name="${NAME_JOINT_4}_motor">
+        <hardwareInterface>hardware_interface/PositionJointInterface</hardwareInterface>
+        <mechanicalReduction>1</mechanicalReduction>
+      </actuator>
+    </transmission>
     <!-- crane_x7_link_4 -->
     <link name="${NAME_LINK_4}">
@@ -270,9 +316,9 @@
       </collision>
       <inertial>
-        <mass value="0.230634"/>
-        <origin xyz="-0.008641 0.083071 -0.000086" rpy="${M_PI} 0 0"/>
-        <inertia ixx="1" ixy="0.0" ixz="0.0"
-          iyy="1" iyz="0.0"
-          izz="1"/>
+        <mass value="0.222"/>
+        <origin xyz="-9.39E-03 6.40E-05 8.04E-02" rpy="${M_PI/2} 0 0"/>
+        <inertia ixx="4.89E-04" ixy="-3.90E-06" ixz="8.29E-08"
+          iyy="1.14E-04" iyz="2.82E-06"
+          izz="5.03E-04"/>
       </inertial>
     </link>
@@ -300,11 +346,4 @@
         </geometry>
       </collision>
-      <inertial>
-        <mass value="0.005"/>
-        <origin xyz="0.000036 0.037855 -0.00018" rpy="${M_PI/2} 0 0"/>
-        <inertia ixx="1" ixy="0.0" ixz="0.0"
-          iyy="1" iyz="0.0"
-          izz="1"/>
-      </inertial>
     </link>
     <!-- crane_x7_joint_cover_4_r -->
@@ -331,11 +370,4 @@
         </geometry>
       </collision>
-      <inertial>
-        <mass value="0.005"/>
-        <origin xyz="0.000036 0.037855 -0.00018" rpy="${M_PI/2} 0 0"/>
-        <inertia ixx="1" ixy="0.0" ixz="0.0"
-          iyy="1" iyz="0.0"
-          izz="1"/>
-      </inertial>
     </link>
     <!-- crane_x7_joint_5 -->
@@ -343,8 +375,23 @@
       <origin xyz="0 0 0.121" rpy="0 0 0"/>
       <axis xyz="0 0 1"/>
-      <limit effort="0.5" velocity="${joints_vlimit}" lower="-2.77343" upper="1.51403"/>
+      <limit effort="4.0" velocity="${joints_vlimit}" lower="-2.77343" upper="1.51403"/>
       <parent link="${NAME_LINK_4}"/>
       <child link="${NAME_LINK_5}"/>
-    </joint>
+      <dynamics damping="0.0" friction="0.0"/>
+    </joint>
+    <!-- For gazebo simulation -->
+    <transmission name="${NAME_JOINT_5}_trans">
+      <provideFeedback>true</provideFeedback>
+      <implicitSpringDamper>0</implicitSpringDamper>
+      <motorTorqueConstant>0.418</motorTorqueConstant>
+      <type>transmission_interface/SimpleTransmission</type>
+      <joint name="${NAME_JOINT_5}">
+        <hardwareInterface>hardware_interface/PositionJointInterface</hardwareInterface>
+      </joint>
+      <actuator name="${NAME_JOINT_5}_motor">
+        <hardwareInterface>hardware_interface/PositionJointInterface</hardwareInterface>
+        <mechanicalReduction>1</mechanicalReduction>
+      </actuator>
+    </transmission>
     <!-- crane_x7_link_5 -->
     <link name="${NAME_LINK_5}">
@@ -365,9 +412,9 @@
       </collision>
       <inertial>
-        <mass value="0.192709"/>
-        <origin xyz="-0.000024 0.001285 0.063837" rpy="0 0 0"/>
-        <inertia ixx="1" ixy="0.0" ixz="0.0"
-          iyy="1" iyz="0.0"
-          izz="1"/>
+        <mass value="0.207"/>
+        <origin xyz="-8.40E-05 4.62E-04 6.37E-02" rpy="0 0 0"/>
+        <inertia ixx="2.90E-04" ixy="1.00E-07" ixz="-4.77E-07"
+          iyy="2.57E-04" iyz="-1.69E-05"
+          izz="8.75E-05"/>
       </inertial>
     </link>
@@ -381,8 +428,23 @@
       <origin xyz="0 0 0.129" rpy="0 0 0"/>
       <axis xyz="0 -1 0"/>
-      <limit effort="0.5" velocity="${joints_vlimit}" lower="-${M_PI/2}" upper="${M_PI/2}"/>
+      <limit effort="4.0" velocity="${joints_vlimit}" lower="-${M_PI/2}" upper="${M_PI/2}"/>
       <parent link="${NAME_LINK_5}"/>
       <child link="${NAME_LINK_6}"/>
-    </joint>
+      <dynamics damping="0.0" friction="0.0"/>
+    </joint>
+    <!-- For gazebo simulation -->
+    <transmission name="${NAME_JOINT_6}_trans">
+      <provideFeedback>true</provideFeedback>
+      <implicitSpringDamper>0</implicitSpringDamper>
+      <motorTorqueConstant>0.418</motorTorqueConstant>
+      <type>transmission_interface/SimpleTransmission</type>
+      <joint name="${NAME_JOINT_6}">
+        <hardwareInterface>hardware_interface/PositionJointInterface</hardwareInterface>
+      </joint>
+      <actuator name="${NAME_JOINT_6}_motor">
+        <hardwareInterface>hardware_interface/PositionJointInterface</hardwareInterface>
+        <mechanicalReduction>1</mechanicalReduction>
+      </actuator>
+    </transmission>
     <!-- crane_x7_link_6 -->
     <link name="${NAME_LINK_6}">
@@ -403,9 +465,9 @@
       </collision>
       <inertial>
-        <mass value="0.130549"/>
-        <origin xyz="0.005713 -0.003707 0.000781" rpy="${M_PI/2} 0 0"/>
-        <inertia ixx="1" ixy="0.0" ixz="0.0"
-          iyy="1" iyz="0.0"
-          izz="1"/>
+        <mass value="0.14"/>
+        <origin xyz="6.10E-03 8.26E-04 -3.55E-03" rpy="${M_PI/2} 0 0"/>
+        <inertia ixx="4.01E-05" ixy="-2.91E-06" ixz="6.39E-07"
+          iyy="6.13E-05" iyz="-4.90E-07"
+          izz="7.35E-05"/>
       </inertial>
     </link>
@@ -414,8 +476,63 @@
       <origin xyz="0 0 0.019" rpy="0 0 0"/>
       <axis xyz="0 0 1"/>
-      <limit effort="0.5" velocity="${joints_vlimit}" lower="-2.96365" upper="2.97132"/>
+      <limit effort="4.0" velocity="${joints_vlimit}" lower="-2.96365" upper="2.97132"/>
       <parent link="${NAME_LINK_6}"/>
       <child link="${end_effector_base_link}"/>
-    </joint>
+      <dynamics damping="0.0" friction="0.0"/>
+    </joint>
+    <!-- For gazebo simulation -->
+    <transmission name="${NAME_JOINT_7}_trans">
+      <provideFeedback>true</provideFeedback>
+      <implicitSpringDamper>0</implicitSpringDamper>
+      <motorTorqueConstant>0.418</motorTorqueConstant>
+      <type>transmission_interface/SimpleTransmission</type>
+      <joint name="${NAME_JOINT_7}">
+        <hardwareInterface>hardware_interface/PositionJointInterface</hardwareInterface>
+      </joint>
+      <actuator name="${NAME_JOINT_7}_motor">
+        <hardwareInterface>hardware_interface/PositionJointInterface</hardwareInterface>
+        <mechanicalReduction>1</mechanicalReduction>
+      </actuator>
+    </transmission>
+    <gazebo>
+      <plugin name='gazebo_ros_control' filename='libgazebo_ros_control.so'>
+        <robotNamespace>/crane_x7</robotNamespace>
+        <robotSimType>gazebo_ros_control/DefaultRobotHWSim</robotSimType>
+        <legacyModeNS>true</legacyModeNS>
+      </plugin>
+    </gazebo>
+    <gazebo reference="${NAME_LINK_BASE}">
+      <material>Gazebo/Red</material>
+    </gazebo>
+    <gazebo reference="${NAME_LINK_1}">
+      <material>Gazebo/White</material>
+    </gazebo>
+    <gazebo reference="${NAME_LINK_2}">
+      <material>Gazebo/White</material>
+    </gazebo>
+    <gazebo reference="${NAME_LINK_3}">
+      <material>Gazebo/White</material>
+    </gazebo>
+    <gazebo reference="${NAME_LINK_4}">
+      <material>Gazebo/White</material>
+    </gazebo>
+    <gazebo reference="${NAME_LINK_5}">
+      <material>Gazebo/White</material>
+    </gazebo>
+    <gazebo reference="${NAME_LINK_6}">
+      <material>Gazebo/White</material>
+    </gazebo>
+    <gazebo reference="${NAME_LINK_COVER_2_L}">
+      <material>Gazebo/Red</material>
+    </gazebo>
+    <gazebo reference="${NAME_LINK_COVER_2_R}">
+      <material>Gazebo/Red</material>
+    </gazebo>
+    <gazebo reference="${NAME_LINK_COVER_4_L}">
+      <material>Gazebo/Red</material>
+    </gazebo>
+    <gazebo reference="${NAME_LINK_COVER_4_R}">
+      <material>Gazebo/Red</material>
+    </gazebo>
   </xacro:macro>
 </robot>

File: crane_x7_description/urdf/crane_x7_mounting_plate.xacro (robot description, xacro)
@@ -27,13 +27,9 @@
         </geometry>
       </collision>
-      <inertial>
-        <mass value="0.001"/>
-        <origin xyz="-0.00669 0.000049 0.017868" rpy="0 0 0"/>
-        <inertia ixx="1.0" ixy="0.0" ixz="0.0"
-          iyy="1.0" iyz="0.0"
-          izz="1.0"/>
-        <mass value="0.387313"/>
-      </inertial>
     </link>
+    <!-- For gazebo simulation -->
+    <gazebo reference="${name}_link">
+      <material>Gazebo/Black</material>
+    </gazebo>
   </xacro:macro>
 </robot>

File: crane_x7_description/urdf/crane_x7_rt_logos.xacro (robot description, xacro)
@@ -14,11 +14,4 @@
         </material>
       </visual>
-      <inertial>
-        <mass value="0"/>
-        <origin xyz="0.000036 0.037855 -0.00018" rpy="${M_PI/2} 0 0"/>
-        <inertia ixx="1" ixy="0.0" ixz="0.0"
-          iyy="1" iyz="0.0"
-          izz="1"/>
-      </inertial>
     </link>
     <joint name="${name}_logo_text_l_joint" type="fixed">
@@ -37,11 +30,4 @@
         <material name="logo_red"/>
       </visual>
-      <inertial>
-        <mass value="0"/>
-        <origin xyz="0.000036 0.037855 -0.00018" rpy="${M_PI/2} 0 0"/>
-        <inertia ixx="1" ixy="0.0" ixz="0.0"
-          iyy="1" iyz="0.0"
-          izz="1"/>
-      </inertial>
     </link>
     <joint name="${name}_logo_symbol_l_joint" type="fixed">
@@ -60,11 +46,4 @@
         <material name="logo_red"/>
       </visual>
-      <inertial>
-        <mass value="0"/>
-        <origin xyz="0.000036 0.037855 -0.00018" rpy="${M_PI/2} 0 0"/>
-        <inertia ixx="1" ixy="0.0" ixz="0.0"
-          iyy="1" iyz="0.0"
-          izz="1"/>
-      </inertial>
     </link>
     <joint name="${name}_logo_text_r_joint" type="fixed">
@@ -83,11 +62,4 @@
         <material name="logo_red"/>
       </visual>
-      <inertial>
-        <mass value="0"/>
-        <origin xyz="0.000036 0.037855 -0.00018" rpy="${M_PI/2} 0 0"/>
-        <inertia ixx="1" ixy="0.0" ixz="0.0"
-          iyy="1" iyz="0.0"
-          izz="1"/>
-      </inertial>
     </link>
     <joint name="${name}_logo_symbol_r_joint" type="fixed">
@@ -96,4 +68,17 @@
       <origin xyz="0 -0.0345 0.065" rpy="0 0 0"/>
     </joint>
+    <!-- For gazebo simulation -->
+    <gazebo reference="${name}_logo_symbol_r_link">
+      <material>Gazebo/Red</material>
+    </gazebo>
+    <gazebo reference="${name}_logo_symbol_l_link">
+      <material>Gazebo/Red</material>
+    </gazebo>
+    <gazebo reference="${name}_logo_text_r_link">
+      <material>Gazebo/Black</material>
+    </gazebo>
+    <gazebo reference="${name}_logo_text_l_link">
+      <material>Gazebo/Black</material>
+    </gazebo>
   </xacro:macro>
 </robot>

File: crane_x7_description/urdf/crane_x7_wide_two_finger_gripper.xacro (robot description, xacro)
@@ -23,9 +23,9 @@
       </collision>
       <inertial>
-        <mass value="0.119807"/>
-        <origin xyz="0.000425 -0.000896 0.018691" rpy="0 0 0"/>
-        <inertia ixx="1" ixy="0.0" ixz="0.0"
-          iyy="1" iyz="0.0"
-          izz="1"/>
+        <mass value="0.121"/>
+        <origin xyz="1.08E-04 -1.03E-03 2.08E-02" rpy="0 0 0"/>
+        <inertia ixx="3.20E-05" ixy="-9.45E-08" ixz="2.61E-07"
+          iyy="4.14E-05" iyz="3.88E-07"
+          izz="4.29E-05"/>
       </inertial>
     </link>
@@ -33,8 +33,23 @@
       <origin xyz="-0.012 0.0 0.024" rpy="0 0 0"/>
       <axis xyz="0 -1 0"/>
-      <limit effort="0.5" velocity="${vlimit}" lower="0.0046" upper="1.62601"/>
+      <limit effort="4.0" velocity="${vlimit}" lower="0.0046" upper="1.62601"/>
       <parent link="${name}_base_link"/>
       <child link="${name}_finger_a_link"/>
+      <dynamics damping="0.0" friction="0.8"/>
     </joint>
+    <!-- for gazebo -->
+    <transmission name="${name}_finger_a_joint_trans">
+      <provideFeedback>true</provideFeedback>
+      <implicitSpringDamper>0</implicitSpringDamper>
+      <motorTorqueConstant>0.418</motorTorqueConstant>
+      <type>transmission_interface/SimpleTransmission</type>
+      <joint name="${name}_finger_a_joint">
+        <hardwareInterface>hardware_interface/PositionJointInterface</hardwareInterface>
+      </joint>
+      <actuator name="${name}_finger_a_joint_motor">
+        <hardwareInterface>hardware_interface/PositionJointInterface</hardwareInterface>
+        <mechanicalReduction>1</mechanicalReduction>
+      </actuator>
+    </transmission>
     <link name="${name}_finger_a_link">
       <visual>
@@ -54,9 +69,9 @@
       </collision>
       <inertial>
-        <mass value="0.015617"/>
-        <origin xyz="-0.002987 0.030318 0.003073" rpy="${M_PI/2} 0 0"/>
-        <inertia ixx="1" ixy="0.0" ixz="0.0"
-          iyy="1" iyz="0.0"
-          izz="1"/>
+        <mass value="0.0158"/>
+        <origin xyz="-2.65E-03 3.54E-03 2.69E-02" rpy="${M_PI/2} 0 0"/>
+        <inertia ixx="1.01E-05" ixy="-1.97E-07" ixz="-9.89E-08"
+        iyy="4.95E-06" iyz="5.37E-07"
+        izz="6.24E-06"/>
       </inertial>
     </link>
@@ -64,8 +79,9 @@
       <origin xyz="0.012 0.0 0.024" rpy="0 0 0"/>
       <axis xyz="0 1 0"/>
-      <limit effort="0.5" velocity="${vlimit}" lower="0.0046" upper="1.62601"/>
+      <limit effort="4.0" velocity="${vlimit}" lower="0.0046" upper="1.62601"/>
       <parent link="${name}_base_link"/>
       <child link="${name}_finger_b_link"/>
       <mimic joint="${name}_finger_a_joint"/>
+      <dynamics damping="0.0" friction="0.8"/>
     </joint>
     <link name="${name}_finger_b_link">
@@ -86,11 +102,28 @@
       </collision>
       <inertial>
-        <mass value="0.014417"/>
-        <origin xyz="0.003058 0.031215 0.002548" rpy="${M_PI/2} 0 0"/>
-        <inertia ixx="1" ixy="0.0" ixz="0.0"
-          iyy="1" iyz="0.0"
-          izz="1"/>
+        <mass value="0.0139"/>
+        <origin xyz="3.01E-03 2.85E-03 3.09E-02" rpy="${M_PI/2} 0 0"/>
+        <inertia ixx="7.48E-06" ixy="3.61E-07" ixz="6.34E-08"
+        iyy="4.09E-06" iyz="2.28E-07"
+        izz="4.37E-06"/>
       </inertial>
     </link>
+    <!-- For gazebo simulation -->
+    <gazebo>
+      <plugin name="crane_x7_gripper_mimic_joint" filename="libroboticsgroup_gazebo_mimic_joint_plugin.so">
+        <joint>${name}_finger_a_joint</joint>
+        <mimicJoint>${name}_finger_b_joint</mimicJoint>
+        <multiplier>1</multiplier>
+      </plugin>
+    </gazebo>
+    <gazebo reference="${name}_base_link">
+      <material>Gazebo/Red</material>
+    </gazebo>
+    <gazebo reference="${name}_finger_a_link">
+      <material>Gazebo/Red</material>
+    </gazebo>
+    <gazebo reference="${name}_finger_b_link">
+      <material>Gazebo/Red</material>
+    </gazebo>
   </xacro:macro>
 </robot>
