Commit message: Correct collision rotation

File: crane_x7_description/urdf/crane_x7_wide_two_finger_gripper.xacro (robot description, xacro)
@@ -47,5 +47,5 @@
       </visual>
       <collision>
-        <origin xyz="0 0 0" rpy="0 0 0"/>
+        <origin xyz="0 0 0" rpy="${M_PI/2} 0 0"/>
         <geometry>
           <mesh filename="package://crane_x7_description/meshes/collision/wide_two_finger_gripper_finger_a.stl"
@@ -79,5 +79,5 @@
       </visual>
       <collision>
-        <origin xyz="0 0 0" rpy="0 0 0"/>
+        <origin xyz="0 0 0" rpy="${M_PI/2} 0 0"/>
         <geometry>
           <mesh filename="package://crane_x7_description/meshes/collision/wide_two_finger_gripper_finger_b.stl"

Commit message: Update URDF parameters

File: crane_x7_description/urdf/crane_x7_wide_two_finger_gripper.xacro (robot description, xacro)
@@ -36,5 +36,5 @@
       <parent link="${name}_base_link"/>
       <child link="${name}_finger_a_link"/>
-      <dynamics damping="1.0e-6" friction="2.0e-1"/>
+      <dynamics damping="1.0e-6" friction="8.0e-1"/>
     </joint>
     <!-- for gazebo -->
@@ -93,5 +93,5 @@
       <child link="${name}_finger_b_link"/>
       <mimic joint="${name}_finger_a_joint"/>
-      <dynamics damping="1.0e-6" friction="2.0e-1"/>
+      <dynamics damping="1.0e-6" friction="8.0e-1"/>
     </joint>
     <link name="${name}_finger_b_link">
