Commit message: Fix dynamics parameters

File: crane_x7_description/urdf/crane_x7_arm.xacro (robot description, xacro)
@@ -84,5 +84,5 @@
       <parent link="${NAME_LINK_BASE}"/>
       <child link="${NAME_LINK_1}"/>
-      <dynamics damping="0.0" friction="0.0"/>
+      <dynamics damping="1.0e-6" friction="2.0e-1"/>
     </joint>
     <!-- For gazebo simulation -->
@@ -142,5 +142,5 @@
       <parent link="${NAME_LINK_1}"/>
       <child link="${NAME_LINK_2}"/>
-      <dynamics damping="0.0" friction="0.0"/>
+      <dynamics damping="1.0e-6" friction="2.0e-1"/>
     </joint>
     <!-- For gazebo simulation -->
@@ -227,5 +227,5 @@
       <parent link="${NAME_LINK_2}"/>
       <child link="${NAME_LINK_3}"/>
-      <dynamics damping="0.0" friction="0.0"/>
+      <dynamics damping="1.0e-6" friction="2.0e-1"/>
     </joint>
     <!-- For gazebo simulation -->
@@ -278,5 +278,5 @@
       <parent link="${NAME_LINK_3}"/>
       <child link="${NAME_LINK_4}"/>
-      <dynamics damping="0.0" friction="0.0"/>
+      <dynamics damping="1.0e-6" friction="2.0e-1"/>
     </joint>
     <!-- For gazebo simulation -->
@@ -360,5 +360,5 @@
       <parent link="${NAME_LINK_4}"/>
       <child link="${NAME_LINK_5}"/>
-      <dynamics damping="0.0" friction="0.0"/>
+      <dynamics damping="1.0e-6" friction="2.0e-1"/>
     </joint>
     <!-- For gazebo simulation -->
@@ -413,5 +413,5 @@
       <parent link="${NAME_LINK_5}"/>
       <child link="${NAME_LINK_6}"/>
-      <dynamics damping="0.0" friction="0.0"/>
+      <dynamics damping="1.0e-6" friction="2.0e-1"/>
     </joint>
     <!-- For gazebo simulation -->
@@ -461,5 +461,5 @@
       <parent link="${NAME_LINK_6}"/>
       <child link="${end_effector_base_link}"/>
-      <dynamics damping="0.0" friction="0.0"/>
+      <dynamics damping="1.0e-6" friction="2.0e-1"/>
     </joint>
     <!-- For gazebo simulation -->
@@ -481,5 +481,5 @@
         <robotNamespace>/crane_x7</robotNamespace>
         <robotSimType>gazebo_ros_control/DefaultRobotHWSim</robotSimType>
-        <legacyModeNS>true</legacyModeNS>
+        <legacyModeNS>false</legacyModeNS>
       </plugin>
     </gazebo>

File: crane_x7_description/urdf/crane_x7_wide_two_finger_gripper.xacro (robot description, xacro)
@@ -36,5 +36,5 @@
       <parent link="${name}_base_link"/>
       <child link="${name}_finger_a_link"/>
-      <dynamics damping="0.0" friction="0.8"/>
+      <dynamics damping="1.0e-6" friction="2.0e-1"/>
     </joint>
     <!-- for gazebo -->
@@ -93,5 +93,5 @@
       <child link="${name}_finger_b_link"/>
       <mimic joint="${name}_finger_a_joint"/>
-      <dynamics damping="0.0" friction="0.8"/>
+      <dynamics damping="1.0e-6" friction="2.0e-1"/>
     </joint>
     <link name="${name}_finger_b_link">

Commit message: Add collision model for joint covers and logos

File: crane_x7_description/urdf/crane_x7_arm.xacro (robot description, xacro)
@@ -199,4 +199,11 @@
         <material name="${shoulder_joint_cover_color}"/>
       </visual>
+      <collision>
+        <origin xyz="0 0 0" rpy="-${M_PI/2} 0 0"/>
+        <geometry>
+          <mesh filename="package://crane_x7_description/meshes/visual/joint_cover.stl"
+              scale="1 1 1"/>
+        </geometry>
+      </collision>
     </link>
     <!-- crane_x7_joint_cover_2_r -->
@@ -216,4 +223,11 @@
         <material name="${shoulder_joint_cover_color}"/>
       </visual>
+      <collision>
+        <origin xyz="0 0 0" rpy="${M_PI/2} 0 0"/>
+        <geometry>
+          <mesh filename="package://crane_x7_description/meshes/visual/joint_cover.stl"
+              scale="1 1 1"/>
+        </geometry>
+      </collision>
     </link>
     <!-- crane_x7_joint_3 -->
@@ -335,4 +349,11 @@
         <material name="${elbow_joint_cover_color}"/>
       </visual>
+      <collision>
+        <origin xyz="0 0 0" rpy="-${M_PI/2} 0 0"/>
+        <geometry>
+          <mesh filename="package://crane_x7_description/meshes/visual/joint_cover.stl"
+              scale="1 1 1"/>
+        </geometry>
+      </collision>
     </link>
     <!-- crane_x7_joint_cover_4_r -->
@@ -352,4 +373,11 @@
         <material name="${elbow_joint_cover_color}"/>
       </visual>
+      <collision>
+        <origin xyz="0 0 0" rpy="${M_PI/2} 0 0"/>
+        <geometry>
+          <mesh filename="package://crane_x7_description/meshes/visual/joint_cover.stl"
+              scale="1 1 1"/>
+        </geometry>
+      </collision>
     </link>
     <!-- crane_x7_joint_5 -->

Commit message: joint5のリミットを左右対称に修正する

File: crane_x7_description/urdf/crane_x7_arm.xacro (robot description, xacro)
@@ -385,5 +385,5 @@
       <origin xyz="0 0 0.121" rpy="0 0 0"/>
       <axis xyz="0 0 1"/>
-      <limit effort="4.0" velocity="${joints_vlimit}" lower="-2.77343" upper="1.51403"/>
+      <limit effort="4.0" velocity="${joints_vlimit}" lower="-2.77343" upper="2.77343"/>
       <parent link="${NAME_LINK_4}"/>
       <child link="${NAME_LINK_5}"/>
